File: hardware/Controller.brd (EAGLE design)
At the start: 38.1 x 58.4 mm, 70 parts, among them Q1 MOSFET-NCHANNEL2N7002PW, Q2 BSS84PW, Q3 BSS84PW, U3 MMA8652FC, U4 MCP6002MS, U5 TXS0101DCK, U6 LCD_1.8, U7 VREG

Commit message: hardware: Change in resistor values in analog section
Parts:
- C12: value 15p -> 470p
- R16, R17: value 1M -> 100k
Changed lines of the file:
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@@
 <attribute name="VALUE" x="35.306" y="6.223" size="1.016" layer="27" font="vector" ratio="14" rot="R180"/>
 </element>
-<element name="R17" library="SparkFun-Resistors" package="0603-RES" value="1M" x="31.75" y="2.54" smashed="yes">
+<element name="R17" library="SparkFun-Resistors" package="0603-RES" value="100k" x="31.75" y="2.54" smashed="yes">
 <attribute name="NAME" x="28.956" y="0.762" size="1.016" layer="25" font="vector" ratio="14"/>
 <attribute name="VALUE" x="30.734" y="1.397" size="1.016" layer="27" font="vector" ratio="14"/>
 </element>
-<element name="R16" library="SparkFun-Resistors" package="0603-RES" value="1M" x="34.29" y="7.62" smashed="yes">
+<element name="R16" library="SparkFun-Resistors" package="0603-RES" value="100k" x="34.29" y="7.62" smashed="yes">
 <attribute name="VALUE" x="33.274" y="6.477" size="1.016" layer="27" font="vector" ratio="14"/>
 </element>
@@
 </element>
 <element name="SH1" library="Parts" package="SHORT_TOP-8" value="SHORT" x="29.210240625" y="15.417934375" smashed="yes" rot="MR90"/>
-<element name="C12" library="SparkFun-Capacitors" package="0603-CAP" value="15p" x="34.29" y="6.35" smashed="yes" rot="R180">
+<element name="C12" library="SparkFun-Capacitors" package="0603-CAP" value="470p" x="34.29" y="6.35" smashed="yes" rot="R180">
 <attribute name="VALUE" x="35.306" y="7.493" size="0.4064" layer="27" font="vector" rot="R180"/>
 </element>
